Commit message: 相机模块添加成功,还没改位置

File: src/ackermann_gazebo/urdf/bot_base.xacro (robot description, xacro)
@@ -243,4 +243,20 @@
         </sensor>
     </gazebo>
+    <link name="camera_link">
+        <visual>
+        <geometry>
+            <box size="0.02 0.05 0.03"/> </geometry>
+        <material name="black"/>
+        </visual>
+        <inertial>
+        <mass value="0.01"/>
+        <inertia ixx="0.0001" ixy="0" ixz="0" iyy="0.0001" iyz="0" izz="0.0001"/>
+        </inertial>
+    </link>
+    <joint name="camera_joint" type="fixed">
+        <parent link="chassis_link"/>
+        <child link="camera_link"/>
+        <origin xyz="0.20 0 ${body_height/2 + 0.015}" rpy="0 0 0"/>
+    </joint>
     <xacro:macro name="wheel_friction" params="link_name">
         <gazebo reference="${link_name}">

File: src/ackermann_gazebo/urdf/gz_ackermann_core.xacro (robot description, xacro)
@@ -28,4 +28,28 @@
     <gazebo reference="virtual_steer_link">
         <material>Gazebo/Yellow</material>
+    </gazebo>
+    <gazebo reference="camera_link">
+        <sensor name="robot_camera" type="camera">
+            <update_rate>60.0</update_rate>
+            <camera name="head">
+                <horizontal_fov>2.61799</horizontal_fov>
+                <image>
+                    <width>1280</width>
+                    <height>720</height>
+                    <format>R8G8B8</format>
+                </image>
+                <clip>
+                    <near>0.02</near>
+                    <far>300</far>
+                </clip>
+            </camera>
+            <plugin name="camera_controller" filename="libgazebo_ros_camera.so">
+                <alwaysOn>true</alwaysOn>
+                <updateRate>0.0</updateRate> <cameraName>robot/camera</cameraName>
+                <imageTopicName>image_raw</imageTopicName>
+                <cameraInfoTopicName>camera_info</cameraInfoTopicName>
+                <frameName>camera_link</frameName>
+            </plugin>
+        </sensor>
     </gazebo>
     <gazebo>

Commit message: 相对位置改好了,但是link名字没在gazebo仿真里面出现

File: src/ackermann_gazebo/urdf/bot_base.xacro (robot description, xacro)
@@ -163,8 +163,8 @@
         <limit effort="200" velocity="100" />
     </joint>
-    <link name="laser_link">
-        <visual>
-            <geometry><cylinder length="0.03" radius="0.025"/></geometry>
-            <origin rpy="0 0 0" xyz="0 0 -0.01"/>
+   <link name="laser_link">
+        <visual>
+            <geometry><cylinder length="0.06" radius="0.025"/></geometry>
+            <origin rpy="0 0 0" xyz="0 0 -0.03"/>
             <material name="white" />
         </visual>
@@ -172,10 +172,11 @@
             <mass value="0.1"/>
             <inertia ixx="0.001" ixy="0.0" ixz="0.0" iyy="0.001" iyz="0.0" izz="0.001"/>
-            <origin xyz="0 0 -0.01"/>
+            <origin xyz="0 0 -0.03"/>
         </inertial>
     </link>
     <joint name="laser_joint" type="fixed">
-        <parent link="chassis_link"/> <child link="laser_link"/>
-        <origin rpy="0 0 0" xyz="0 0 ${body_height/2 + 0.02}"/>
+        <parent link="chassis_link"/>
+        <child link="laser_link"/>
+        <origin rpy="0 0 0" xyz="0 0 ${body_height/2 + 0.05}"/>
     </joint>
     <gazebo reference="laser_link">

Commit message: 名字可以显示

File: src/ackermann_gazebo/urdf/bot_base.xacro (robot description, xacro)
@@ -248,5 +248,7 @@
         <geometry>
             <box size="0.02 0.05 0.03"/> </geometry>
-        <material name="black"/>
+        <material name="red">
+            <color rgba="1.0 0.0 0.0 1.0" />
+        </material>
         </visual>
         <inertial>

File: src/ackermann_gazebo/urdf/gz_ackermann_core.xacro (robot description, xacro)
@@ -30,4 +30,5 @@
     </gazebo>
     <gazebo reference="camera_link">
+        <material>Gazebo/Red</material>
         <sensor name="robot_camera" type="camera">
             <update_rate>60.0</update_rate>
@@ -123,3 +124,12 @@
         <limit lower="-3.14" upper="3.14" effort="200" velocity="20" />
     </joint>
+    <gazebo reference="laser_joint">
+        <preserveFixedJoint>true</preserveFixedJoint>
+    </gazebo>
+    <gazebo reference="imu_joint">
+        <preserveFixedJoint>true</preserveFixedJoint>
+    </gazebo>
+    <gazebo reference="camera_joint">
+        <preserveFixedJoint>true</preserveFixedJoint>
+    </gazebo>
 </robot>
